File: Elec/ReceiverBoard/ReceiverBoard.kicad_pcb (KiCad board)
At the start: 2 copper layers, 40 x 100 mm, 2 parts, among them J1 Conn_01x03, J2 Conn_01x03

Commit message: SUKU ReceiverBoard created
Parts:
- added J3: Conn_01x03, suku_basics:BATTERY_2X_18650, B.Cu at (80.0, 90.0)
- added J4: Conn_01x03, suku_basics:SERVO_MICRO, F.Cu at (100.0, 185.0)
- moved J2 102.0 mm to (120.0, 90.0)
- moved J1 15.0 mm to (100.0, 105.0), turned to 180 degrees
Connections:
- J1 pad 1: (no net) -> /ORANGE
- J1 pad 2: (no net) -> /RED
- J1 pad 3: (no net) -> /BLACK
Other:
- board size 40 x 100 mm -> 70 x 175 mm

Commit message: SUKU sync
Parts:
- added H1: MountingHole, MountingHole:MountingHole_2.1mm, F.Cu at (87.5, 37.5)
- added H10: MountingHole, MountingHole:MountingHole_2.1mm, F.Cu at (132.5, 130.0)
- added H11: MountingHole, MountingHole:MountingHole_2.1mm, F.Cu at (92.5, 52.5)
- added H12: MountingHole, MountingHole:MountingHole_2.1mm, F.Cu at (107.5, 52.5)
- added H13: MountingHole, MountingHole:MountingHole_2.1mm, F.Cu at (67.5, 207.5)
- added H14: MountingHole, MountingHole:MountingHole_2.1mm, F.Cu at (132.5, 207.5)
- added H2: MountingHole, MountingHole:MountingHole_2.1mm, F.Cu at (112.5, 37.5)
- added H3: MountingHole, MountingHole:MountingHole_2.1mm, F.Cu at (67.5, 47.5)
- added H4: MountingHole, MountingHole:MountingHole_2.1mm, F.Cu at (132.5, 47.5)
- added H5: MountingHole, MountingHole:MountingHole_2.1mm, F.Cu at (92.5, 47.5)
- added H6: MountingHole, MountingHole:MountingHole_2.1mm, F.Cu at (107.5, 47.5)
- added H7: MountingHole, MountingHole:MountingHole_2.1mm, F.Cu at (67.5, 52.5)
- added H8: MountingHole, MountingHole:MountingHole_2.1mm, F.Cu at (132.5, 52.5)
- added H9: MountingHole, MountingHole:MountingHole_2.1mm, F.Cu at (67.5, 130.0)
